File: ControlBoard_Hardware/ControlBoard_Hardware.kicad_sch (KiCad schematic)
At the start: 51 parts, among them U10 MCP1415, U11 TSR_1-2450, U2 TSR_1-2450, U3 MCP1415, U4 OKI-78SR-12, U6 MCP1415, U7 MCP1415, U8 MCP1415, U9 MCP1415

Commit message: finished board layour
Parts:
- removed H4: MountingHole, MountingHole:MountingHole_3.2mm_M3, symbol Mechanical:MountingHole
- added D5: LED, LED_SMD:LED_0603_1608Metric_Pad1.05x0.95mm_HandSolder, symbol Device:LED
- added R6: 300, Resistor_SMD:R_0603_1608Metric_Pad0.98x0.95mm_HandSolder, symbol Device:R
Connections:
- net Input_PWR is gone; now on net PWR_IN: R1.1
- net +5V: now also U1.47 (Vin); no longer U1. (Vin)
- net +5VA: now also R6.1
- net Discharge_Toggle: now also U1.11 (MOSI); no longer U1.12 (MISO)
- net GND: now also U1.44 (GND), U1.45 (GND), D5.1 (K); no longer U1. (Vin)
- net Relay_Toggle: now also U1.12 (MISO); no longer U1.11 (MOSI)
- net Safety Switch: now also U1.15 (A1); no longer U1.16 (A2)
- net Trigger Signal: now also U1.16 (A2); no longer U1.15 (A1)
- net +3.3V renamed +3V3
- net +3V3: now also U1.46 (3V3)
- new net: D5.2 (A), R6.2
- no-connect marks 0 -> 6

Commit message: ahhhhhhhh
Parts:
- removed PowerSwich1: Molex_SL_02, MRDT_Connectors:MOLEX_SL_02_Horizontal, symbol MRDT_Connectors:Molex_SL_02
Connections:
- net +5VA: now also C14.1
- net LED Data: no longer C14.1
- net PWR_IN: now also Conn1.2
Changed lines of the file:
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@@
   (junction (at 111.76 43.18) (diameter 0) (color 0 0 0 0)
   )
-  (junction (at 246.38 25.4) (diameter 0) (color 0 0 0 0)
-  )
   (junction (at 83.82 171.45) (diameter 0) (color 0 0 0 0)
   )
@@
   )
   (junction (at 69.85 49.53) (diameter 0) (color 0 0 0 0)
+  )
+  (junction (at 256.54 22.86) (diameter 0) (color 0 0 0 0)
   )
   (junction (at 36.83 52.07) (diameter 0) (color 0 0 0 0)
@@
   (no_connect (at 242.57 125.73))
   (no_connect (at 242.57 128.27))
-  (wire (pts (xy 243.84 25.4) (xy 246.38 25.4))
+  (wire (pts (xy 243.84 25.4) (xy 247.65 25.4))
     (stroke (width 0) (type default))
   )
@@
     (stroke (width 0) (type default))
   )
-  (wire (pts (xy 31.75 26.67) (xy 36.83 26.67))
+  (wire (pts (xy 25.4 26.67) (xy 36.83 26.67))
     (stroke (width 0) (type default))
   )
@@
     (stroke (width 0) (type default))
   )
-  (wire (pts (xy 246.38 25.4) (xy 247.65 25.4))
-    (stroke (width 0) (type default))
-  )
   (wire (pts (xy 83.82 175.26) (xy 83.82 171.45))
     (stroke (width 0) (type default))
@@
     (stroke (width 0) (type default))
   )
-  (wire (pts (xy 246.38 25.4) (xy 246.38 26.67))
-    (stroke (width 0) (type default))
-  )
   (wire (pts (xy 40.64 77.47) (xy 36.83 77.47))
     (stroke (width 0) (type default))
@@
     (stroke (width 0) (type default))
   )
+  (wire (pts (xy 246.38 22.86) (xy 256.54 22.86))
+    (stroke (width 0) (type default))
+  )
   (wire (pts (xy 204.47 22.86) (xy 204.47 20.32))
     (stroke (width 0) (type default))
@@
     (stroke (width 0) (type default))
   )
-  (wire (pts (xy 25.4 26.67) (xy 29.21 26.67))
+  (wire (pts (xy 246.38 26.67) (xy 246.38 22.86))
     (stroke (width 0) (type default))
   )
@@
     )
   )
-  (symbol (lib_id "MRDT_Connectors:Molex_SL_02") (at 33.02 21.59 90) (unit 1)
-    (in_bom yes) (on_board yes) (dnp no)
-    (property "Reference" "PowerSwich1" (at 25.4 15.24 90)
-      (effects (font (size 1.524 1.524)) (justify right))
-    )
-    (property "Value" "Molex_SL_02" (at 25.4 17.78 90)
-      (effects (font (size 1.524 1.524)) (justify right))
-    )
-    (property "Footprint" "MRDT_Connectors:MOLEX_SL_02_Horizontal" (at 35.56 21.59 0)
-      (effects (font (size 1.524 1.524)) hide)
-    )
-    (property "Datasheet" "" (at 35.56 21.59 0)
-      (effects (font (size 1.524 1.524)) hide)
-    )
-    (pin "1")
-    (pin "2")
-    (instances
-      (project "ControlBoard_Hardware"
-        (path "/487df2d1-0681-470c-8e27-af1d48fa6afe"
-          (reference "PowerSwich1") (unit 1)
-        )
-      )
-    )
-  )
   (symbol (lib_id "MRDT_Connectors:Molex_SL_02") (at 130.81 57.15 0) (unit 1)
     (in_bom yes) (on_board yes) (dnp no) (fields_autoplaced)
@@
       (effects (font (size 1.27 1.27)) hide)
     )
-    (pin "46")
-    (pin "44")
-    (pin "45")
-    (pin "47")
     (pin "0")
     (pin "1")
@@
     (pin "3")
     (pin "4")
+    (pin "44")
+    (pin "45")
+    (pin "46")
+    (pin "47")
     (pin "5")
     (pin "6")
