File: ControlBoard_Hardware/ControlBoard_Hardware.kicad_sch (KiCad schematic)
At the start: 51 parts, among them U10 MCP1415, U11 TSR_1-2450, U2 TSR_1-2450, U3 MCP1415, U4 OKI-78SR-12, U6 MCP1415, U7 MCP1415, U8 MCP1415, U9 MCP1415

Commit message: yes
Parts:
- C10, C12, C2, C4, C6, C8: value 10uF -> 1uF
Changed lines of the file:
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@@
       (effects (font (size 1.27 1.27)))
     )
-    (property "Value" "10uF" (at 78.7463 167.64 90)
+    (property "Value" "1uF" (at 78.7463 167.64 90)
       (effects (font (size 1.27 1.27)))
     )
@@
       (effects (font (size 1.27 1.27)))
     )
-    (property "Value" "10uF" (at 120.6563 130.81 90)
+    (property "Value" "1uF" (at 120.6563 130.81 90)
       (effects (font (size 1.27 1.27)))
     )
@@
       (effects (font (size 1.27 1.27)))
     )
-    (property "Value" "10uF" (at 78.7463 130.81 90)
+    (property "Value" "1uF" (at 78.7463 130.81 90)
       (effects (font (size 1.27 1.27)))
     )
@@
       (effects (font (size 1.27 1.27)))
     )
-    (property "Value" "10uF" (at 36.8363 167.64 90)
+    (property "Value" "1uF" (at 36.8363 167.64 90)
       (effects (font (size 1.27 1.27)))
     )
@@
       (effects (font (size 1.27 1.27)))
     )
-    (property "Value" "10uF" (at 120.6563 167.64 90)
+    (property "Value" "1uF" (at 120.6563 167.64 90)
       (effects (font (size 1.27 1.27)))
     )
@@
       (effects (font (size 1.27 1.27)))
     )
-    (property "Value" "10uF" (at 36.8363 130.81 90)
-      (effects (font (size 1.27 1.27)))
-    )
+    (property "Value" "1uF" (at 36.8363 130.81 90)
+      (effects (font (size 1.27 1.27)))
+    )
